File: tiny1616_dev_board.kicad_pcb (KiCad board)
At the start: 2 copper layers, 47.6 x 29.5 mm, 33 parts, among them J1 Barrel_Jack, J2 USB_C_Receptacle_USB2.0, J3 Conn_02x03_Odd_Even, J4 Conn_01x02_Female, J5 Conn_01x09_Male, J6 Conn_01x09_Male, U1 AMS1117-5.0, U2 ATtiny1616-M, U3 CH340G, U4 MAX3485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

Commit message: README
Parts:
- added G***: LOGO, Local footprints:qr-code, B.Cu at (92.7, 58.6)
